File: PSU_Standalone/PSU_Standalone.sch (KiCad schematic (older format))
At the start: 22 parts

Commit message: Added first two CMCs
Parts:
- removed J?: Conn_01x02_Female, symbol Connector:Conn_01x02_Female
- added C?: 1u, Capacitor_THT:C_Disc_D3.0mm_W1.6mm_P2.50mm, symbol Device:CP
- added D?: D_Schottky, symbol Device:D_Schottky
- added J2: Conn_01x03_Male, Connector_PinHeader_2.54mm:PinHeader_1x03_P2.54mm_Vertical, symbol Connector:Conn_01x03_Male
- C1, C2, C3, C4, C5: renamed from C?; footprint (none) -> Capacitor_THT:C_Disc_D3.0mm_W1.6mm_P2.50mm
- FL1: renamed from FL?; footprint (none) -> Bamboulibs:CYSMB100805TL-4T-701R Common Mode Choke
- FL2: renamed from FL?; footprint (none) -> Bamboulibs:FL2D-30-222 Common Mode Choke
- J1: renamed from J?; footprint (none) -> Connector_PinHeader_2.54mm:PinHeader_1x02_P2.54mm_Vertical
- Q1: renamed from Q?; footprint (none) -> Package_TO_SOT_THT:TO-220-3_Horizontal_TabDown
- R1, R2, R3, R4, R5, R6, R7, R8: renamed from R?; footprint (none) -> Resistor_THT:R_Axial_DIN0411_L9.9mm_D3.6mm_P12.70mm_Horizontal
- RV1: renamed from RV?; footprint (none) -> nixies:Chinese Pots
- T1: renamed from T?; footprint (none) -> Bamboulibs:Transformer_LPR6235
- U1: renamed from U?; footprint (none) -> Package_SO:SOIC-8_3.9x4.9mm_P1.27mm
- gave numbers to parts that had none: 1
Connections:
- net T_Sec_Hi is gone; now on net T_Prim_Lo: FL1.4, FL2.4, FL3.4, T1.2 (AB)
- net GND: now also C?.2, J2.3 (Pin_3)
- net HV: now also D?.1 (K), J2.2 (Pin_2); no longer R2.2, RV1.1
- net T_Prim_Lo: now also Q1.2 (D)
- net T_Sec_Lo: now also T1.3 (SA), C?.1, D?.2 (A); no longer T1.1 (AA)
- net VCC: now also FL1.2, FL2.2, FL3.2, T1.1 (AA)
- removed net T_Prim_Hi: FL1.2, FL2.2, FL3.2, T1.3 (SA)
- new net FBK: J2.1 (Pin_1), R2.2, RV1.1

Commit message: Did board design
Parts:
- added F1: Cut to enable external feedback, Bamboulibs:Cut_trace, symbol Device:Fuse
- C4: footprint Capacitor_THT:C_Disc_D3.0mm_W1.6mm_P2.50mm -> Capacitor_THT:CP_Radial_D4.0mm_P1.50mm
- C5: footprint Capacitor_THT:C_Disc_D3.0mm_W1.6mm_P2.50mm -> Capacitor_THT:CP_Radial_D5.0mm_P2.00mm
- C6: renamed from C?; footprint Capacitor_THT:C_Disc_D3.0mm_W1.6mm_P2.50mm -> Capacitor_THT:CP_Radial_D6.3mm_P2.50mm
- D1: renamed from D?; footprint (none) -> Diode_THT:D_DO-41_SOD81_P10.16mm_Horizontal
- FL1: value EMI_Filter_CommonMode -> CYSMB100805TL-4T-701R
- FL2: value EMI_Filter_CommonMode -> FL2D-30-222
- FL3: value EMI_Filter_CommonMode -> Dummy for future use; footprint (none) -> Bamboulibs:Transformer_dummy
- J1: value Conn_01x02_Male -> Vin
- J2: value Conn_01x03_Male -> Vout
Connections:
- net FBK: now also F1.2
- net HV: now also F1.1
Changed lines of the file:
@@
 P 800 1000
 F 0 "J1" H 908 1181 50  0000 C CNN
-F 1 "Conn_01x02_Male" H 908 1090 50  0000 C CNN
+F 1 "Vin" H 908 1090 50  0000 C CNN
 F 2 "Connector_PinHeader_2.54mm:PinHeader_1x02_P2.54mm_Vertical" H 800 1000 50  0001 C CNN
 F 3 "~" H 800 1000 50  0001 C CNN
@@
 F 0 "C4" H 8615 1796 50  0000 L CNN
 F 1 "10u" H 8615 1705 50  0000 L CNN
-F 2 "Capacitor_THT:C_Disc_D3.0mm_W1.6mm_P2.50mm" H 8538 1600 50  0001 C CNN
+F 2 "Capacitor_THT:CP_Radial_D4.0mm_P1.50mm" H 8538 1600 50  0001 C CNN
 F 3 "~" H 8500 1750 50  0001 C CNN
 	1    8500 1750
@@
 F 0 "C5" H 9118 1796 50  0000 L CNN
 F 1 "220u" H 9118 1705 50  0000 L CNN
-F 2 "Capacitor_THT:C_Disc_D3.0mm_W1.6mm_P2.50mm" H 9038 1600 50  0001 C CNN
+F 2 "Capacitor_THT:CP_Radial_D5.0mm_P2.00mm" H 9038 1600 50  0001 C CNN
 F 3 "~" H 9000 1750 50  0001 C CNN
 	1    9000 1750
@@
 P 2250 5000
 F 0 "FL1" H 2250 4675 50  0000 C CNN
-F 1 "EMI_Filter_CommonMode" H 2250 4766 50  0000 C CNN
+F 1 "CYSMB100805TL-4T-701R" H 2250 4766 50  0000 C CNN
 F 2 "Bamboulibs:CYSMB100805TL-4T-701R Common Mode Choke" H 2250 5040 50  0001 C CNN
 F 3 "~" H 2250 5040 50  0001 C CNN
@@
 P 5250 5000
 F 0 "FL2" H 5250 4675 50  0000 C CNN
-F 1 "EMI_Filter_CommonMode" H 5250 4766 50  0000 C CNN
+F 1 "FL2D-30-222" H 5250 4766 50  0000 C CNN
 F 2 "Bamboulibs:FL2D-30-222 Common Mode Choke" H 5250 5040 50  0001 C CNN
 F 3 "~" H 5250 5040 50  0001 C CNN
@@
 P 8250 5000
 F 0 "FL3" H 8250 4675 50  0000 C CNN
-F 1 "EMI_Filter_CommonMode" H 8250 4766 50  0000 C CNN
-F 2 "" H 8250 5040 50  0001 C CNN
+F 1 "Dummy for future use" H 8250 4766 50  0000 C CNN
+F 2 "Bamboulibs:Transformer_dummy" H 8250 5040 50  0001 C CNN
 F 3 "~" H 8250 5040 50  0001 C CNN
 	1    8250 5000
@@
 P 10700 1000
 F 0 "J2" H 10672 1024 50  0000 R CNN
-F 1 "Conn_01x03_Male" H 10672 933 50  0000 R CNN
+F 1 "Vout" H 10672 933 50  0000 R CNN
 F 2 "Connector_PinHeader_2.54mm:PinHeader_1x03_P2.54mm_Vertical" H 10700 1000 50  0001 C CNN
 F 3 "~" H 10700 1000 50  0001 C CNN
@@
 HV
 $Comp
-L Device:CP C?
+L Device:CP C6
 U 1 1 5EA614E6
 P 9500 3750
-F 0 "C?" H 9618 3796 50  0000 L CNN
+F 0 "C6" H 9618 3796 50  0000 L CNN
 F 1 "1u" H 9618 3705 50  0000 L CNN
-F 2 "Capacitor_THT:C_Disc_D3.0mm_W1.6mm_P2.50mm" H 9538 3600 50  0001 C CNN
+F 2 "Capacitor_THT:CP_Radial_D6.3mm_P2.50mm" H 9538 3600 50  0001 C CNN
 F 3 "~" H 9500 3750 50  0001 C CNN
 	1    9500 3750
@@
 $EndComp
 $Comp
-L Device:D_Schottky D?
+L Device:D_Schottky D1
 U 1 1 5EA626E9
 P 10000 3500
-F 0 "D?" H 10000 3284 50  0000 C CNN
+F 0 "D1" H 10000 3284 50  0000 C CNN
 F 1 "D_Schottky" H 10000 3375 50  0000 C CNN
-F 2 "" H 10000 3500 50  0001 C CNN
+F 2 "Diode_THT:D_DO-41_SOD81_P10.16mm_Horizontal" H 10000 3500 50  0001 C CNN
 F 3 "~" H 10000 3500 50  0001 C CNN
 	1    10000 3500
@@
 $EndComp
 $Comp
-L power:GND #PWR?
+L power:GND #PWR0115
 U 1 1 5EA62F64
 P 9500 4000
-F 0 "#PWR?" H 9500 3750 50  0001 C CNN
+F 0 "#PWR0115" H 9500 3750 50  0001 C CNN
 F 1 "GND" H 9505 3827 50  0000 C CNN
 F 2 "" H 9500 4000 50  0001 C CNN
@@
 	10150 3500 10500 3500
 $Comp
-L power:VCC #PWR?
+L power:VCC #PWR0116
 U 1 1 5EA6C9CF
 P 7800 3000
-F 0 "#PWR?" H 7800 2850 50  0001 C CNN
+F 0 "#PWR0116" H 7800 2850 50  0001 C CNN
 F 1 "VCC" V 7817 3128 50  0000 L CNN
 F 2 "" H 7800 3000 50  0001 C CNN
@@
 Wire Wire Line
 	7800 3000 8000 3000
+Text GLabel 8750 900  0    50   Input ~ 0
+FBK
+Text GLabel 9250 900  2    50   Input ~ 0
+HV
+$Comp
+L Device:Fuse F1
+U 1 1 5EACCE07
+P 9000 900
+F 0 "F1" V 8803 900 50  0000 C CNN
+F 1 "Cut to enable external feedback" V 8894 900 50  0000 C CNN
+F 2 "Bamboulibs:Cut_trace" V 8930 900 50  0001 C CNN
+F 3 "~" H 9000 900 50  0001 C CNN
+	1    9000 900
+	0    1    1    0
+$EndComp
+Wire Wire Line
+	8850 900  8750 900
+Wire Wire Line
+	9150 900  9250 900
 $EndSCHEMATC
